File: revC-fm/Avionics.kicad_sch (KiCad schematic)
At the start: 70 parts, among them J1 5031821852, P2 TSM-105-01-F-SV, P3 FTSH-105-01-F-DV-K-TR, SW1 KMR231NG LFS, SW2 KMR231NG LFS, U4 MAX708RESA-T, U5 imu-stamp-revA, U6 SN74LVC1T45DCK, U7 MR25H40MDF, U8 ATSAMD51N20A-AUT, Y1 32.768kHz

Commit message: changed RF connector to TH
Parts:
- added BT1: 2998, SierraLobo:BatteryHolder_Keystone_2998_1x6.8mm, symbol Device:Battery_Cell
- added C137: 0.1uF, Capacitor_SMD:C_0603_1608Metric, symbol Device:C
- added R268, R271: 10k, Resistor_SMD:R_0603_1608Metric, symbol Device:R_US
- added U45: DS1343D-33+, Package_DFN_QFN:DFN-14-1EP_3x3mm_P0.4mm_EP1.78x2.35mm, symbol SierraLobo:DS1343D-33+
- added Y2: 32.768kHz, SierraLobo:Crystal_SMD_3215-2Pin_3.2x1.5mm, symbol Device:Crystal
- U7: footprint SierraLobo:SON127P600X500X90-9N -> Package_DFN_QFN:DFN-8-1EP_6x5mm_P1.27mm_EP2x2mm
- Y1: footprint Crystal:Crystal_SMD_3215-2Pin_3.2x1.5mm -> SierraLobo:Crystal_SMD_3215-2Pin_3.2x1.5mm
- renumbered LED2 to LED1, LED1 to LED2, LED4 to LED3, LED3 to LED4, R271 to R23, R23 to R24, R24 to R25, R25 to R26, R26 to R27, R27 to R28, R28 to R29
Connections:
- net 3.3V: now also C137.1, R268.1, U45.14 (VCC)
- net GND: now also BT1.2 (-), C137.2, U45.15 (EP), U45.7 (GND)
- net PC20 renamed RTC_CE
- net RTC_CE: now also R271.1
- new net: U45.2 (X1), Y2.1
- new net: U45.3 (X2), Y2.2
- new net: R271.2, U45.8 (CE)
- new net: BT1.1 (+), U45.1 (VBAT)
- new net: R268.2, U45.13 (SERMODE)
- new net MISO_RTC: U45.11 (SDO)
- new net MOSI_RTC: U45.10 (SDI)
- new net SCK_RTC: U45.9 (SCLK)
- no-connect marks 8 -> 11
Other:
- note added: "6.8mm coin cell"
- note added: "RTC"
- note removed: "NOTE: Components labeled "do not install" (DNI) are not populated by default"
- moved on the sheet: C25, J1, P2, P3, R11, R14, R16, R20, U5
