File: revC-fm/Bus_Protection.kicad_sch (KiCad schematic)
At the start: 2 parts, among them Q71 MMBT3904T

Commit message: working
Parts:
- renumbered R94 to R67
Changed lines of the file:
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@@
   (symbol (lib_id "Device:R_US") (at 177.8 135.89 270) (unit 1)
     (in_bom yes) (on_board yes) (dnp no)
-    (property "Reference" "R94" (at 177.8 130.683 90)
+    (property "Reference" "R67" (at 177.8 130.683 90)
       (effects (font (size 1.27 1.27)))
     )
@@
       (project "mainboard"
         (path "/d1441985-7b63-4bf8-a06d-c70da2e3b78b/00000000-0000-0000-0000-00005ede7915"
-          (reference "R94") (unit 1)
+          (reference "R67") (unit 1)
         )
       )
@@
         )
         (path "/d1441985-7b63-4bf8-a06d-c70da2e3b78b/00000000-0000-0000-0000-00005ede7915"
-          (reference "Q3") (unit 1)
+          (reference "Q11") (unit 1)
         )
       )
@@
   (symbol (lib_id "power:GND") (at 189.23 140.97 0) (unit 1)
     (in_bom yes) (on_board yes) (dnp no)
-    (property "Reference" "#PWR0104" (at 189.23 147.32 0)
+    (property "Reference" "#PWR090" (at 189.23 147.32 0)
       (effects (font (size 1.27 1.27)) hide)
     )
@@
       (project "mainboard"
         (path "/d1441985-7b63-4bf8-a06d-c70da2e3b78b/00000000-0000-0000-0000-00005ede7915"
-          (reference "#PWR0104") (unit 1)
+          (reference "#PWR090") (unit 1)
         )
       )
