File: revC-fm/db_led.kicad_sch (KiCad schematic)
At the start: 3 parts, among them Q73 MUN5311DW1

Commit message: working
Parts:
- removed D5: YEL, LED_SMD:LED_0402_1005Metric, symbol Device:LED
- removed R68: 1.8k, Resistor_SMD:R_0402_1005Metric, symbol Device:R_US
Other:
- note removed: "1.85V, 20mcd, 2mA"
Changed lines of the file:
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@@
-    (stroke (width 0) (type default))
-  )
-  (wire (pts (xy 161.29 57.15) (xy 161.29 60.96))
     (stroke (width 0) (type default))
   )
@@
     (stroke (width 0) (type default))
   )
-  (wire (pts (xy 161.29 68.58) (xy 161.29 71.12))
-    (stroke (width 0) (type default))
-  )
   (wire (pts (xy 151.13 86.36) (xy 146.05 86.36))
-    (stroke (width 0) (type default))
-  )
-  (wire (pts (xy 157.48 57.15) (xy 161.29 57.15))
     (stroke (width 0) (type default))
   )
   (wire (pts (xy 129.54 86.36) (xy 135.89 86.36))
     (stroke (width 0) (type default))
-  )
-  (text "1.85V, 20mcd, 2mA\n\n\n" (at 170.18 82.55 0)
-    (effects (font (size 1.27 1.27)) (justify left bottom))
   )
   (global_label "LED_EN" (shape output) (at 129.54 96.52 180) (fields_autoplaced)
@@
     )
   )
-  (global_label "LED_PWR" (shape input) (at 157.48 57.15 180) (fields_autoplaced)
-    (effects (font (size 1.016 1.016)) (justify right))
-    (property "Intersheetrefs" "${INTERSHEET_REFS}" (at 148.9538 57.15 0)
-      (effects (font (size 1.016 1.016)) (justify right) hide)
-    )
-  )
   (hierarchical_label "ON" (shape input) (at 129.54 86.36 180) (fields_autoplaced)
     (effects (font (size 1.27 1.27)) (justify right))
-  )
-  (symbol (lib_id "Device:LED") (at 161.29 74.93 90) (unit 1)
-    (in_bom yes) (on_board yes) (dnp no) (fields_autoplaced)
-    (property "Reference" "D5" (at 165.1 75.8825 90)
-      (effects (font (size 1.27 1.27)) (justify right))
-    )
-    (property "Value" "YEL" (at 165.1 78.4225 90)
-      (effects (font (size 1.27 1.27)) (justify right))
-    )
-    (property "Footprint" "LED_SMD:LED_0402_1005Metric" (at 161.29 74.93 0)
-      (effects (font (size 1.27 1.27)) hide)
-    )
-    (property "Datasheet" "https://www.kingbrightusa.com/images/catalog/SPEC/APHHS1005LSYCK-J3-PF.pdf" (at 161.29 74.93 0)
-      (effects (font (size 1.27 1.27)) hide)
-    )
-    (property "Mfr. Part No" "APHHS1005LSYCK/J3-PF" (at 161.29 74.93 0)
-      (effects (font (size 1.27 1.27)) hide)
-    )
-    (pin "1")
-    (pin "2")
-    (instances
-      (project "mainboard"
-        (path "/d1441985-7b63-4bf8-a06d-c70da2e3b78b/00000000-0000-0000-0000-00005cec5dde/a78437db-a0fc-4cde-8346-4d17e2576807"
-          (reference "D5") (unit 1)
-        )
-        (path "/d1441985-7b63-4bf8-a06d-c70da2e3b78b/00000000-0000-0000-0000-00005cec5dde"
-          (reference "LED5") (unit 1)
-        )
-        (path "/d1441985-7b63-4bf8-a06d-c70da2e3b78b/94774350-68be-4131-9d22-bdea2eae3261/26c7b1e9-b366-492c-be9e-83b88a5fa8e6"
-          (reference "LED5") (unit 1)
-        )
-        (path "/d1441985-7b63-4bf8-a06d-c70da2e3b78b/94774350-68be-4131-9d22-bdea2eae3261/51f684eb-7c47-4469-82a8-b507e037a52f"
-          (reference "LED11") (unit 1)
-        )
-        (path "/d1441985-7b63-4bf8-a06d-c70da2e3b78b/94774350-68be-4131-9d22-bdea2eae3261/14a6998c-ffe6-42d1-963e-e80449405007"
-          (reference "LED12") (unit 1)
-        )
-        (path "/d1441985-7b63-4bf8-a06d-c70da2e3b78b/94774350-68be-4131-9d22-bdea2eae3261/bdd3e858-dbd7-4a4f-b8ee-98b758544d47"
-          (reference "LED13") (unit 1)
-        )
-        (path "/d1441985-7b63-4bf8-a06d-c70da2e3b78b/94774350-68be-4131-9d22-bdea2eae3261/1da642f5-94f2-4bd1-98ca-462c89216b58"
-          (reference "LED9") (unit 1)
-        )
-        (path "/d1441985-7b63-4bf8-a06d-c70da2e3b78b/94774350-68be-4131-9d22-bdea2eae3261/0355bb7f-4ca3-4b4d-a29e-300b0aa4ccec"
-          (reference "LED10") (unit 1)
-        )
-      )
-    )
   )
   (symbol (lib_id "power:GND") (at 161.29 96.52 0) (unit 1)
@@
         (path "/d1441985-7b63-4bf8-a06d-c70da2e3b78b/94774350-68be-4131-9d22-bdea2eae3261/51f684eb-7c47-4469-82a8-b507e037a52f"
           (reference "#PWR0189") (unit 1)
-        )
-        (path "/d1441985-7b63-4bf8-a06d-c70da2e3b78b/94774350-68be-4131-9d22-bdea2eae3261/14a6998c-ffe6-42d1-963e-e80449405007"
-          (reference "#PWR0190") (unit 1)
-        )
-        (path "/d1441985-7b63-4bf8-a06d-c70da2e3b78b/94774350-68be-4131-9d22-bdea2eae3261/bdd3e858-dbd7-4a4f-b8ee-98b758544d47"
-          (reference "#PWR0191") (unit 1)
-        )
-        (path "/d1441985-7b63-4bf8-a06d-c70da2e3b78b/94774350-68be-4131-9d22-bdea2eae3261/1da642f5-94f2-4bd1-98ca-462c89216b58"
-          (reference "#PWR0156") (unit 1)
-        )
-        (path "/d1441985-7b63-4bf8-a06d-c70da2e3b78b/94774350-68be-4131-9d22-bdea2eae3261/0355bb7f-4ca3-4b4d-a29e-300b0aa4ccec"
-          (reference "#PWR0179") (unit 1)
         )
       )
@@
           (reference "Q74") (unit 1)
         )
-        (path "/d1441985-7b63-4bf8-a06d-c70da2e3b78b/94774350-68be-4131-9d22-bdea2eae3261/14a6998c-ffe6-42d1-963e-e80449405007"
-          (reference "Q70") (unit 1)
-        )
-        (path "/d1441985-7b63-4bf8-a06d-c70da2e3b78b/94774350-68be-4131-9d22-bdea2eae3261/bdd3e858-dbd7-4a4f-b8ee-98b758544d47"
-          (reference "Q72") (unit 1)
-        )
-        (path "/d1441985-7b63-4bf8-a06d-c70da2e3b78b/94774350-68be-4131-9d22-bdea2eae3261/1da642f5-94f2-4bd1-98ca-462c89216b58"
-          (reference "Q63") (unit 1)
-        )
-        (path "/d1441985-7b63-4bf8-a06d-c70da2e3b78b/94774350-68be-4131-9d22-bdea2eae3261/0355bb7f-4ca3-4b4d-a29e-300b0aa4ccec"
-          (reference "Q73") (unit 1)
-        )
       )
     )
@@
           (reference "Q74") (unit 2)
         )
-        (path "/d1441985-7b63-4bf8-a06d-c70da2e3b78b/94774350-68be-4131-9d22-bdea2eae3261/14a6998c-ffe6-42d1-963e-e80449405007"
-          (reference "Q70") (unit 2)
-        )
-        (path "/d1441985-7b63-4bf8-a06d-c70da2e3b78b/94774350-68be-4131-9d22-bdea2eae3261/bdd3e858-dbd7-4a4f-b8ee-98b758544d47"
-          (reference "Q72") (unit 2)
-        )
-        (path "/d1441985-7b63-4bf8-a06d-c70da2e3b78b/94774350-68be-4131-9d22-bdea2eae3261/1da642f5-94f2-4bd1-98ca-462c89216b58"
-          (reference "Q63") (unit 2)
-        )
-        (path "/d1441985-7b63-4bf8-a06d-c70da2e3b78b/94774350-68be-4131-9d22-bdea2eae3261/0355bb7f-4ca3-4b4d-a29e-300b0aa4ccec"
-          (reference "Q73") (unit 2)
-        )
       )
-    )
-  )
-  (symbol (lib_id "Device:R_US") (at 161.29 64.77 180) (unit 1)
-    (in_bom yes) (on_board yes) (dnp no) (fields_autoplaced)
-    (property "Reference" "R68" (at 163.83 64.135 0)
-      (effects (font (size 1.27 1.27)) (justify right))
-    )
-    (property "Value" "1.8k" (at 163.83 66.675 0)
-      (effects (font (size 1.27 1.27)) (justify right))
-    )
-    (property "Footprint" "Resistor_SMD:R_0402_1005Metric" (at 160.274 64.516 90)
-      (effects (font (size 1.27 1.27)) hide)
-    )
-    (property "Datasheet" "~" (at 161.29 64.77 0)
-      (effects (font (size 1.27 1.27)) hide)
-    )
-    (property "Mfr. Part No" "" (at 161.29 64.77 0)
-      (effects (font (size 1.27 1.27)) hide)
-    )
-    (pin "1")
-    (pin "2")
-    (instances
-      (project "mainboard"
-        (path "/d1441985-7b63-4bf8-a06d-c70da2e3b78b/00000000-0000-0000-0000-00005cec5dde/a78437db-a0fc-4cde-8346-4d17e2576807"
-          (reference "R68") (unit 1)
-        )
-        (path "/d1441985-7b63-4bf8-a06d-c70da2e3b78b/00000000-0000-0000-0000-00005cec5dde"
-          (reference "R41") (unit 1)
-        )
-        (path "/d1441985-7b63-4bf8-a06d-c70da2e3b78b/94774350-68be-4131-9d22-bdea2eae3261/26c7b1e9-b366-492c-be9e-83b88a5fa8e6"
-          (reference "R41") (unit 1)
-        )
-        (path "/d1441985-7b63-4bf8-a06d-c70da2e3b78b/94774350-68be-4131-9d22-bdea2eae3261/51f684eb-7c47-4469-82a8-b507e037a52f"
-          (reference "R43") (unit 1)
-        )
-        (path "/d1441985-7b63-4bf8-a06d-c70da2e3b78b/94774350-68be-4131-9d22-bdea2eae3261/14a6998c-ffe6-42d1-963e-e80449405007"
-          (reference "R272") (unit 1)
-        )
-        (path "/d1441985-7b63-4bf8-a06d-c70da2e3b78b/94774350-68be-4131-9d22-bdea2eae3261/bdd3e858-dbd7-4a4f-b8ee-98b758544d47"
-          (reference "R273") (unit 1)
-        )
-        (path "/d1441985-7b63-4bf8-a06d-c70da2e3b78b/94774350-68be-4131-9d22-bdea2eae3261/1da642f5-94f2-4bd1-98ca-462c89216b58"
-          (reference "R178") (unit 1)
-        )
-        (path "/d1441985-7b63-4bf8-a06d-c70da2e3b78b/94774350-68be-4131-9d22-bdea2eae3261/0355bb7f-4ca3-4b4d-a29e-300b0aa4ccec"
-          (reference "R180") (unit 1)
-        )
-      )
