File: revC-fm/5V_regulator.kicad_sch (KiCad schematic)
At the start: 17 parts, among them U18 TPS630701RNMR

Commit message: working
Parts:
- added C38: 0.1uF, Capacitor_SMD:C_0402_1005Metric, symbol Device:C
- added D5: YEL, LED_SMD:LED_0402_1005Metric, symbol Device:LED
- added Q73: MUN5311DW1, Package_TO_SOT_SMD:SOT-363_SC-70-6, symbol SierraLobo:MUN5312DW1
- added R32: 10mR, Resistor_SMD:R_1206_3216Metric, symbol Device:R_US
- added R68: 1.8k, Resistor_SMD:R_0402_1005Metric, symbol Device:R_US
- added U12: INA230AIRGTR, SierraLobo:INA230AIRGTR, symbol SierraLobo:INA230AxRGT
- renumbered C60 to C41, C61 to C42, C62 to C43, C63 to C44, C64 to C45, C65 to C46, C66 to C47, C67 to C48, C68 to C49, L4 to L3, R58 to R43, R59 to R44, R267 to R45, R61 to R46, R270 to R47, U18 to U13
Connections:
- net PG: now also Q73.4 (E1)
- net VOUT: now also R32.1, U12.11 (Vbus), U12.12 (Vin-); no longer C45.1, C46.1, C47.1, C48.1, R256.1, R45.1, U13.7 (VOUT)
- net GND renamed EP
- net EP: now also C38.2, Q73.1 (E2), U12.10 (GND), U12.17 (EP)
- new net: D5.2 (A), R68.1
- new net: Q73.2 (B2), Q73.3 (C1)
- new net: D5.1 (K), Q73.6 (C2)
- new net 3.3V: C38.1, U12.9 (VS)
- new net A0: U12.2 (A0)
- new net A1: U12.1 (A1)
- new net LED_EN: Q73.5 (B1)
- new net LED_PWR: R68.2
- new net SCL_PWR: U12.5 (SCL)
- new net SDA_PWR: U12.4 (SDA)
- new net VOUT_SEN: C45.1, C46.1, C47.1, C48.1, R256.1, R32.2, R45.1, U12.13 (Vin+), U13.7 (VOUT)
- no-connect marks 0 -> 2
Other:
- note added: "decide address"
- moved on the sheet: C41, C42, C43, C44, C45, C46, C47, C48, C49, L3, R256, R43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

Commit message: almost done!!!!!
Parts:
- renumbered D5 to LED5, R68 to R41
Connections:
- net VIO is gone; now on net 3.3V: R46.1
- net VBUS_IN renamed VIN_PROT
- no-connect marks 2 -> 1
Other:
- sheet OCP ports: added none; removed VIO
- note added: "INPUT: VBUS 5-8.4V"
- note added: "Indicator LED"
- note added: "OUTPUT: 5V, 2A (max, 10W)"
- note added: "Output Power Monitor"
- note added: "PARAMATERS"
- note removed: "Heirarchal Pin Descriptions: EN = enables PFET before regulator ~{ALERT} = OCP alert, turns off PFET, toggle LATCH to clear LATCH = assign normally high, pull low to clear alert LIMIT = OCP trip setting resistor."
- note removed: "payload / rf regulator based from TI WebBench Design"
- moved on the sheet: C38, C41, C42, C43, C44, C45, C46, C47, C48, C49, L3, LED5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
