File: revC-fm/5V_regulator.kicad_sch (KiCad schematic)
At the start: 23 parts, among them Q73 MUN5311DW1, U12 INA230AIRGTR, U13 TPS630701RNMR

Commit message: updated fab files
Parts:
- C38: Manufacturer (none) -> TDK; Mfr. Part No (none) -> CGA2B3X7R1H104K050BE
- C73: renamed from C45; Manufacturer (none) -> Murata
- C74: renamed from C46; Manufacturer (none) -> Murata
- C75: renamed from C47; Manufacturer (none) -> Murata
- C76: renamed from C48; Manufacturer (none) -> Murata
- C77: renamed from C41; Manufacturer (none) -> TDK
- C78: renamed from C42; Manufacturer (none) -> TDK
- C79: renamed from C43; Manufacturer (none) -> TDK
- C80: renamed from C44; Manufacturer (none) -> Murata
- C82: renamed from C49; Manufacturer (none) -> TDK; Mfr. Part No (none) -> CGA2B3X7R1H104K050BE
- L6: renamed from L3; Manufacturer (none) -> Würth Elektronik
- LED5: Manufacturer (none) -> Kingbright; Mfr. Part No (none) -> APHHS1005LSYCK/J3-PF
- Q73: Manufacturer (none) -> onsemi; Mfr. Part No (none) -> MUN5311DW1
- R136: renamed from R43; Manufacturer (none) -> Stackpole Electronics; Mfr. Part No (none) -> RMCF0402FT1M00
- R137: renamed from R44; Manufacturer (none) -> Stackpole Electronics; Mfr. Part No (none) -> RMCF0402FT1M00
- R138: renamed from R45; Manufacturer (none) -> Stackpole Electronics; Mfr. Part No (none) -> RMCF0603ZT0R00
- R140: renamed from R46; Manufacturer (none) -> Stackpole Electronics; Mfr. Part No (none) -> RMCF0402FT1M00
- R256: Manufacturer (none) -> Stackpole Electronics; Mfr. Part No (none) -> RMCF0402FT100K
- R32: Manufacturer (none) -> Vishay Dale; Mfr. Part No (none) -> WSLP1206R0100
- R41: value 1.8k -> 1.5k; Manufacturer (none) -> Stackpole Electronics; Mfr. Part No (none) -> RMCF0402FT1K50
- U12: Manufacturer (none) -> Texas Instruments
- U20: renamed from U13; Manufacturer (none) -> Texas Instruments
- renumbered R47 to R139
Other:
- sheet OCP ports: added IN, OUT; removed VIN, VOUT

Commit message: updated per review, improved docs
Parts:
- removed Q73: MUN5311DW1, Package_TO_SOT_SMD:SOT-363_SC-70-6, symbol SierraLobo:MUN5312DW1
- added Q18: MMDT3946, Package_TO_SOT_SMD:SOT-363_SC-70-6, symbol Transistor_BJT:MMDT3946
- added R5: 100k, Resistor_SMD:R_0402_1005Metric, symbol Device:R_US
- added R91: 10k, Resistor_SMD:R_0402_1005Metric, symbol Device:R_US
- added TP1 (x2): RCU-0C, SierraLobo:TestPoint_TE_RCU_0603, symbol Connector:TestPoint
- R142: renamed from R136; value 1Meg -> 100k; Mfr. Part No RMCF0402FT1M00 -> RMCF0402FT100K
- R143: renamed from R137; value 1Meg -> 100k; Mfr. Part No RMCF0402FT1M00 -> RMCF0402FT100K
- R146: renamed from R139; Manufacturer (none) -> N/A; Mfr. Part No (none) -> N/A
- R147: renamed from R140; value 1Meg -> 100k; Mfr. Part No RMCF0402FT1M00 -> RMCF0402FT100K
- renumbered C73 to C74, C74 to C75, C75 to C76, C76 to C77, C77 to C78, C78 to C79, C79 to C80, C80 to C81, C82 to C83, R138 to R144
Connections:
- net EP: now also Q18.1 (E1), R91.1
- net LED_EN: now also Q18.5 (B2)
- net PG: now also R5.2
- net VIN_PROT: now also TP1.1
- net VOUT: now also TP1.1
- net at U12.3 (~{Alert}): now also R91.2
- net at LED5.1 (K): now also Q18.6 (C1)
- new net: Q18.2 (B1), Q18.3 (C2)
- new net: Q18.4 (E2), R5.1
- no-connect marks 1 -> 0
Other:
- note removed: "decide address"
- moved on the sheet: R142, R143
