File: revC-fm/analog_cond.kicad_sch (KiCad schematic)
At the start: 19 parts, among them U29 DG4052E, U30 DG4051E, U31 LT6004CMS8#PBF

Commit message: routing
Parts:
- C129: renamed from C117; footprint Capacitor_SMD:C_0402_1005Metric -> Capacitor_SMD:C_0603_1608Metric
- C130: renamed from C115; footprint Capacitor_SMD:C_0402_1005Metric -> Capacitor_SMD:C_0603_1608Metric
- C131: renamed from C116; footprint Capacitor_SMD:C_0402_1005Metric -> Capacitor_SMD:C_0603_1608Metric
- C132: renamed from C118; footprint Capacitor_SMD:C_0402_1005Metric -> Capacitor_SMD:C_0603_1608Metric
- RN1: footprint SierraLobo:RAVF164D -> Resistor_SMD:R_Array_Convex_4x0402
- renumbered R228 to R217, R225 to R218, R226 to R219, R229 to R220, R227 to R221, R231 to R222, R230 to R223, R233 to R224, R224 to R225, R232 to R226, U31 to U32, U29 to U33, U30 to U34

Commit message: changed RF connector to TH
Parts:
- renumbered C129 to C119, C130 to C120, C131 to C121, C132 to C122, R217 to R213, R218 to R214, R219 to R215, R220 to R216, R221 to R217, R222 to R218, R223 to R219, R224 to R220, R225 to R221, R226 to R222, U32 to U30, U33 to U31, U34 to U32

Commit message: working revC review changes
Parts:
- renumbered C119 to C120, C120 to C121, C121 to C122, C122 to C123, R213 to R230, R214 to R231, R215 to R232, R216 to R233, R217 to R234, R218 to R235, R219 to R236, R220 to R237, R221 to R238, R222 to R239, U30 to U31, U31 to U32, U32 to U33

Commit message: working revC
Parts:
- removed R238: 0, Resistor_SMD:R_0603_1608Metric, symbol Device:R_US
- added C26 (x2): 0.1uF, Capacitor_SMD:C_0402_1005Metric, symbol Device:C
- added R136, R62: 232k, Resistor_SMD:R_0603_1608Metric, symbol Device:R_US
- added R137, R63: 33k, Resistor_SMD:R_0603_1608Metric, symbol Device:R_US
- C112: renamed from C120; footprint Capacitor_SMD:C_0603_1608Metric -> Capacitor_SMD:C_0402_1005Metric
- C113: renamed from C121; footprint Capacitor_SMD:C_0603_1608Metric -> Capacitor_SMD:C_0402_1005Metric
- C114: renamed from C122; footprint Capacitor_SMD:C_0603_1608Metric -> Capacitor_SMD:C_0402_1005Metric
- RN1: Mfr. Part No (none) -> RAVF164DJT1K00
- U32: renamed from U31; Mfr. Part No (none) -> LT6004CMS8#PBF
- U33: renamed from U32; Mfr. Part No (none) -> DG4052EEN-T1-GE4
- U34: renamed from U33; Mfr. Part No (none) -> DG4051EEN-T1-GE4
- renumbered C123 to C115, R230 to R182, R231 to R183, R232 to R184, R233 to R185, R234 to R186, R235 to R187, R236 to R188, R237 to R189, R239 to R190
Connections:
- net BATT_NTC: now also U34.15 (X4)
- net GND: now also C26.2, C26.2, R137.2, R63.2
- net SOLAR_TLE_HI: no longer names the net of U34.13 (X2)
- net SOLAR_TLE_HI: now also C26.1, R62.2, R63.1
- net SOLAR_TLE_LO: no longer names the net of U34.10 (X3)
- net SOLAR_TLE_LO: now also C26.1, R136.2, R137.1
- new net SOLAR_1: R62.1
- new net SOLAR_2: R136.1
Other:
- note added: "3.3V MAX"
- note added: "MCP9700 Temperature Sensors"
- note added: "MUX 1: NTC and TEMP sensors"
- note added: "Vsolar 24Vin MAX Set max input 3V"
- note removed: "MUX 1: NTC and TEMP sensors 4:1 x2"
- note removed: "all analog signals have a max of 3.3V."
- moved on the sheet: C112, C114, C115, R187, R188, R189, R190, RN1, U32B, U32C, U34

Commit message: working
Parts:
- renumbered C113 to C92, C112 to C93, C114 to C94, C115 to C97, R182 to R145, R183 to R146, R184 to R147, R185 to R148, R186 to R149, R187 to R150, R62 to R151, R136 to R152, R188 to R153, R189 to R154, R63 to R155, R137 to R156, R190 to R157, U32 to U29, U33 to U30, U34 to U31

Commit message: almost done!!!!!
Parts:
- added C134: 10nF, Capacitor_SMD:C_0603_1608Metric, symbol Device:C
Connections:
- net NTC: now also C134.2
- net at R147.2, R148.1, R149.2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: now also C134.1
Other:
- note added: "See TI App Note SBOA323"
- note removed: "See TI App Note xxxx"
Changed lines of the file:
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@@
   (junction (at 137.16 52.07) (diameter 0) (color 0 0 0 0)
+  )
+  (junction (at 179.07 74.93) (diameter 0) (color 0 0 0 0)
   )
   (junction (at 121.92 135.89) (diameter 0) (color 0 0 0 0)
@@
     (stroke (width 0) (type default))
   )
+  (wire (pts (xy 156.21 86.36) (xy 162.56 86.36))
+    (stroke (width 0) (type default))
+  )
   (wire (pts (xy 147.32 52.07) (xy 147.32 48.26))
     (stroke (width 0) (type default))
@@
     (stroke (width 0) (type default))
   )
+  (wire (pts (xy 156.21 74.93) (xy 156.21 86.36))
+    (stroke (width 0) (type default))
+  )
   (wire (pts (xy 179.07 54.61) (xy 190.5 54.61))
     (stroke (width 0) (type default))
@@
     (stroke (width 0) (type default))
   )
+  (wire (pts (xy 170.18 86.36) (xy 179.07 86.36))
+    (stroke (width 0) (type default))
+  )
   (wire (pts (xy 222.25 49.53) (xy 236.22 49.53))
     (stroke (width 0) (type default))
@@
   )
   (wire (pts (xy 237.49 116.84) (xy 264.16 116.84))
+    (stroke (width 0) (type default))
+  )
+  (wire (pts (xy 179.07 86.36) (xy 179.07 74.93))
     (stroke (width 0) (type default))
   )
@@
     (effects (font (size 1.27 1.27)) (justify left bottom))
   )
-  (text "See TI App Note xxxx" (at 152.4 39.37 0)
+  (text "See TI App Note SBOA323" (at 152.4 39.37 0)
     (effects (font (size 1.27 1.27)) (justify left bottom))
   )
@@
         (path "/d1441985-7b63-4bf8-a06d-c70da2e3b78b/cda1ad7d-3729-4e28-9f04-75ded2a9befd"
           (reference "#SUPPLY035") (unit 1)
+        )
+      )
+    )
+  )
+  (symbol (lib_id "Device:C") (at 166.37 86.36 90) (unit 1)
+    (in_bom yes) (on_board yes) (dnp no) (fields_autoplaced)
+    (property "Reference" "C134" (at 166.37 80.01 90)
+      (effects (font (size 1.27 1.27)))
+    )
+    (property "Value" "10nF" (at 166.37 82.55 90)
+      (effects (font (size 1.27 1.27)))
+    )
+    (property "Footprint" "Capacitor_SMD:C_0603_1608Metric" (at 170.18 85.3948 0)
+      (effects (font (size 1.27 1.27)) hide)
+    )
+    (property "Datasheet" "~" (at 166.37 86.36 0)
+      (effects (font (size 1.27 1.27)) hide)
+    )
+    (property "Mfr. Part No" "" (at 166.37 86.36 0)
+      (effects (font (size 1.27 1.27)) hide)
+    )
+    (pin "1")
+    (pin "2")
+    (instances
+      (project "mainboard"
+        (path "/d1441985-7b63-4bf8-a06d-c70da2e3b78b/cda1ad7d-3729-4e28-9f04-75ded2a9befd"
+          (reference "C134") (unit 1)
         )
       )
@@
     (instances
       (project "mainboard"
-        (path "/d1441985-7b63-4bf8-a06d-c70da2e3b78b/00000000-0000-0000-0000-00005cec5dde/a78437db-a0fc-4cde-8346-4d17e2576807" (page "20"))
         (path "/d1441985-7b63-4bf8-a06d-c70da2e3b78b/cda1ad7d-3729-4e28-9f04-75ded2a9befd" (page "18"))
       )
@@
     (instances
       (project "mainboard"
-        (path "/d1441985-7b63-4bf8-a06d-c70da2e3b78b/00000000-0000-0000-0000-00005cec5dde/a78437db-a0fc-4cde-8346-4d17e2576807" (page "20"))
         (path "/d1441985-7b63-4bf8-a06d-c70da2e3b78b/cda1ad7d-3729-4e28-9f04-75ded2a9befd" (page "3"))
       )
@@
     (instances
       (project "mainboard"
-        (path "/d1441985-7b63-4bf8-a06d-c70da2e3b78b/00000000-0000-0000-0000-00005cec5dde/a78437db-a0fc-4cde-8346-4d17e2576807" (page "20"))
         (path "/d1441985-7b63-4bf8-a06d-c70da2e3b78b/cda1ad7d-3729-4e28-9f04-75ded2a9befd" (page "20"))
       )
@@
     (instances
       (project "mainboard"
-        (path "/d1441985-7b63-4bf8-a06d-c70da2e3b78b/00000000-0000-0000-0000-00005cec5dde/a78437db-a0fc-4cde-8346-4d17e2576807" (page "20"))
         (path "/d1441985-7b63-4bf8-a06d-c70da2e3b78b/cda1ad7d-3729-4e28-9f04-75ded2a9befd" (page "21"))
       )
