File: revC-fm/analog_cond.kicad_sch (KiCad schematic)
At the start: 25 parts, among them U29 LT6004CMS8#PBF, U30 DG4052E, U31 DG4051E

Commit message: updated fab files
Parts:
- C105: renamed from C92; Manufacturer (none) -> TDK; Mfr. Part No (none) -> CGA2B3X7R1H104K050BE
- C106: renamed from C93; Manufacturer (none) -> TDK; Mfr. Part No (none) -> CGA2B3X7R1H104K050BE
- C107: renamed from C134; Manufacturer (none) -> TDK; Mfr. Part No (none) -> CGA3E2X7R1H103K080AE
- C108: renamed from C94; Manufacturer (none) -> TDK; Mfr. Part No (none) -> CGA2B3X7R1H104K050BE
- C111: renamed from C97; Manufacturer (none) -> TDK; Mfr. Part No (none) -> CGA3E2X7R1H103K080AE
- C26: Manufacturer (none) -> TDK; Mfr. Part No (none) -> CGA2B3X7R1H104K050BE
- R238: renamed from R145; Manufacturer (none) -> Stackpole Electronics; Mfr. Part No (none) -> RMCF0603ZT0R00
- R239: renamed from R146; value R_US -> 10k; Manufacturer (none) -> Stackpole Electronics; Mfr. Part No (none) -> RMCF0603FT10K0
- R240: renamed from R147; value R_US -> DNP; now not fitted
- R241: renamed from R148; value R_US -> 10k; Manufacturer (none) -> Stackpole Electronics; Mfr. Part No (none) -> RMCF0603FT10K0
- R242: renamed from R149; value R_US -> DNP; now not fitted
- R243: renamed from R150; Manufacturer (none) -> Stackpole Electronics; Mfr. Part No (none) -> RMCF0603ZT0R00
- R244: renamed from R151; Manufacturer (none) -> Stackpole Electronics; Mfr. Part No RMCF0603FT226K -> RMCF0402FT232K
- R245: renamed from R152; Manufacturer (none) -> Stackpole Electronics; Mfr. Part No RMCF0603FT226K -> RMCF0402FT232K
- R246: renamed from R153; Manufacturer (none) -> Stackpole Electronics; Mfr. Part No (none) -> RMCF0603FT110K
- R247: renamed from R154; Manufacturer (none) -> Stackpole Electronics; Mfr. Part No (none) -> RMCF0603FG1K00
- R248: renamed from R155; Manufacturer (none) -> Stackpole Electronics; Mfr. Part No (none) -> RMCF0603FT33K0
- R249: renamed from R156; Manufacturer (none) -> Stackpole Electronics; Mfr. Part No (none) -> RMCF0603FT33K0
- R250: renamed from R157; Manufacturer (none) -> Stackpole Electronics; Mfr. Part No (none) -> RMCF0603FT110K
- RN1: Manufacturer (none) -> Stackpole Electronics
- U29: Manufacturer (none) -> Analog Devices
- U30, U31: Manufacturer (none) -> Vishay Siliconix
Other:
- note added: "See TI App Note SBOA323 if tuning desired."
- note removed: "See TI App Note SBOA323"

Commit message: updated per review, improved docs
Parts:
- R250: renamed from R240; Manufacturer (none) -> N/A; Mfr. Part No (none) -> N/A
- R252: renamed from R242; Manufacturer (none) -> N/A; Mfr. Part No (none) -> N/A
- R254: renamed from R244; Mfr. Part No RMCF0402FT232K -> RMCF0603FT232K
- R255: renamed from R245; Mfr. Part No RMCF0402FT232K -> RMCF0603FT232K
- renumbered C105 to C106, C106 to C107, C107 to C108, C108 to C109, C111 to C112, R238 to R248, R239 to R249, R241 to R251, R243 to R253, R246 to R256, R247 to R257, R248 to R258, R249 to R259, R250 to R260
