File: revC-fm/ocp_detector.kicad_sch (KiCad schematic)
At the start: 14 parts, among them Q21 BSZ180P03NS3GATMA1, Q34 MMDT3946, U45 INA300AIDSQT

Commit message: changed RF connector to TH
Parts:
- renumbered C144 to C134, R257 to R253, R258 to R254, R34 to R255, R259 to R256, R260 to R257, U45 to U43

Commit message: working revC review changes
Parts:
- added R271: 1k, Resistor_SMD:R_0603_1608Metric, symbol Device:R_US
- R36: value 10mR -> 22mR
- renumbered C134 to C135, D18 to D17, R253 to R270, R254 to R272, R255 to R273, R256 to R274, R257 to R275, U43 to U44
Connections:
- net ~{ALERT}: now also R271.2; no longer U44.5 (~{ALERT})
- new net: R271.1, U44.5 (~{ALERT})
Other:
- note added: "Inhibit Closed = EN high & ~{ALERT} low"
- note added: "VTrip = 18mV delay = 100us hyst = 8mV"
- note removed: "100us delay"
- note removed: "8mV hys"
- note removed: "ITrip = 1.8A VTrip = 18mV delay = 100us"
- moved on the sheet: R270, RN7B

Commit message: working revC
Parts:
- removed Q21: BSZ180P03NS3GATMA1, SierraLobo:PG-TSDSON-8_3.3x3.3mm, symbol SierraLobo:BSZ086
- removed R273: 1k, Resistor_SMD:R_0603_1608Metric, symbol Device:R_US
- C146: footprint Capacitor_SMD:C_0603_1608Metric -> Capacitor_SMD:C_0402_1005Metric
- Q21: Mfr. Part No (none) -> BSZ180P03NS3GATMA1
- Q34: Mfr. Part No (none) -> MMDT3946-7-F
- R256: renamed from R270; footprint Resistor_SMD:R_0603_1608Metric -> Resistor_SMD:R_0402_1005Metric
- R257: renamed from R271; footprint Resistor_SMD:R_0603_1608Metric -> Resistor_SMD:R_0402_1005Metric
- R258: renamed from R272; footprint Resistor_SMD:R_0603_1608Metric -> Resistor_SMD:R_0402_1005Metric
- R259: renamed from R274; footprint Resistor_SMD:R_0603_1608Metric -> Resistor_SMD:R_0402_1005Metric
- R260: renamed from R275; footprint Resistor_SMD:R_0603_1608Metric -> Resistor_SMD:R_0402_1005Metric
- R36: footprint Resistor_SMD:R_0805_2012Metric -> Resistor_SMD:R_1206_3216Metric; Mfr. Part No (none) -> WSLPx
- RN7: Mfr. Part No (none) -> RAVF164DJT1K00
- U37: renamed from U44; Mfr. Part No (none) -> INA300AIDSQT
- renumbered C135 to C129, D17 to D14
Connections:
- net GND: now also U37.11 (EP)
Other:
- note added: "10 can be higher?"

Commit message: working
Parts:
- renumbered C129 to C111, D14 to D20, Q34 to Q5, Q21 to Q59, R256 to R221, R257 to R222, R258 to R223, R259 to R224, R260 to R225, U37 to U34

Commit message: almost done!!!!!
Parts:
- Q59: value BSZ180P03NS3GATMA1 -> BSZ180
Connections:
- net VIN renamed IN
- net VIO renamed 3.3V
- net VOUT renamed OUT
Other:
- note added: "10k iffyish"
- note added: "Heirarchal Pin Descriptions: EN = enables PFET before regulator ~{ALERT} = OCP alert, turns off PFET, toggle LATCH to clear LATCH = MCU assigns normally high, toggle to clear alert LIMIT = OCP trip setting resistor."
- note added: "Output = EN high & ~{ALERT} low"
- note added: "Output Control"
- note added: "Output Switch"
- note added: "Overcurrent Detector / Latch"
- note added: "Overcurrent Protection"
- note removed: "10 can be higher?"
- note removed: "Inhibit Closed = EN high & ~{ALERT} low"
- moved on the sheet: C111, C146, D20, Q59, Q5A, Q5B, R221, R222, R223, R224, R225, R36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
