File: revC-fm/leds.kicad_sch (KiCad schematic)
At the start: 22 parts, among them P2 TSM-102-01-L-SV-P-TR, Q20 MMBT3906T, Q71 MMBT3904T, U6 SN74LVC1T45DCK

Commit message: working
Parts:
- renumbered Q20 to Q53
Other:
- removed sheet LED1
- removed sheet LED2
- removed sheet LED3
- removed sheet LED4
- removed sheet LED5
- removed sheet LED6
- note removed: "Discrete LEDs"
- moved on the sheet: C28, C30, C31, C32, C33, LED1, LED2, LED3, LED4, P2, Q53, Q71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

Commit message: almost done!!!!!
Parts:
- renumbered R68 to R269, R68 to R55
Changed lines of the file:
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@@
   (symbol (lib_id "power:GND") (at 123.19 74.93 0) (unit 1)
     (in_bom yes) (on_board yes) (dnp no)
-    (property "Reference" "#PWR0108" (at 123.19 81.28 0)
+    (property "Reference" "#PWR0187" (at 123.19 81.28 0)
       (effects (font (size 1.27 1.27)) hide)
     )
@@
     (instances
       (project "mainboard"
-        (path "/d1441985-7b63-4bf8-a06d-c70da2e3b78b/00000000-0000-0000-0000-00005cec5dde/a78437db-a0fc-4cde-8346-4d17e2576807"
-          (reference "#PWR0108") (unit 1)
-        )
         (path "/d1441985-7b63-4bf8-a06d-c70da2e3b78b/00000000-0000-0000-0000-00005cec5dde"
           (reference "#PWR0187") (unit 1)
@@
   (symbol (lib_id "Device:R_US") (at 58.42 97.79 90) (mirror x) (unit 1)
     (in_bom yes) (on_board yes) (dnp no)
-    (property "Reference" "R68" (at 58.42 102.87 90)
+    (property "Reference" "R269" (at 58.42 102.87 90)
       (effects (font (size 1.27 1.27)))
     )
@@
     (instances
       (project "mainboard"
-        (path "/d1441985-7b63-4bf8-a06d-c70da2e3b78b/00000000-0000-0000-0000-00005cec5dde/a78437db-a0fc-4cde-8346-4d17e2576807"
-          (reference "R68") (unit 1)
-        )
         (path "/d1441985-7b63-4bf8-a06d-c70da2e3b78b/00000000-0000-0000-0000-00005cec5dde"
           (reference "R269") (unit 1)
@@
   (symbol (lib_id "Device:R_US") (at 123.19 55.88 180) (unit 1)
     (in_bom yes) (on_board yes) (dnp yes) (fields_autoplaced)
-    (property "Reference" "R68" (at 125.73 55.245 0)
+    (property "Reference" "R55" (at 125.73 55.245 0)
       (effects (font (size 1.27 1.27)) (justify right))
     )
@@
     (instances
       (project "mainboard"
-        (path "/d1441985-7b63-4bf8-a06d-c70da2e3b78b/00000000-0000-0000-0000-00005cec5dde/a78437db-a0fc-4cde-8346-4d17e2576807"
-          (reference "R68") (unit 1)
-        )
         (path "/d1441985-7b63-4bf8-a06d-c70da2e3b78b/00000000-0000-0000-0000-00005cec5dde"
           (reference "R55") (unit 1)
@@
   (symbol (lib_id "Device:R_US") (at 111.76 67.31 90) (unit 1)
     (in_bom yes) (on_board yes) (dnp no) (fields_autoplaced)
-    (property "Reference" "R68" (at 111.76 62.23 90)
+    (property "Reference" "R269" (at 111.76 62.23 90)
       (effects (font (size 1.27 1.27)))
     )
@@
     (instances
       (project "mainboard"
-        (path "/d1441985-7b63-4bf8-a06d-c70da2e3b78b/00000000-0000-0000-0000-00005cec5dde/a78437db-a0fc-4cde-8346-4d17e2576807"
-          (reference "R68") (unit 1)
-        )
         (path "/d1441985-7b63-4bf8-a06d-c70da2e3b78b/00000000-0000-0000-0000-00005cec5dde"
           (reference "R269") (unit 1)

Commit message: updated fab files
Parts:
- added R138: 0, Resistor_SMD:R_0603_1608Metric, symbol Device:R_US
- C28, C30, C31, C32, C33: Manufacturer (none) -> TDK; Mfr. Part No (none) -> CGA2B3X7R1H104K050BE
- LED1, LED2, LED3, LED4: Manufacturer (none) -> Adafruit
- P2: Manufacturer (none) -> Samtec
- Q69: renamed from Q53; Manufacturer (none) -> Diodes Incorporated
- Q71: Manufacturer (none) -> Diodes Incorporated
- R17, R20, R21, R26, R27: Manufacturer (none) -> Panasonic; Mfr. Part No (none) -> ERJ-2GEJ102X
- R17: Manufacturer (none) -> Stackpole Electronics; Mfr. Part No (none) -> RMCF0603ZT0R00
- R269, R55: Manufacturer (none) -> Stackpole Electronics; Mfr. Part No (none) -> RMCF0402FT10K0
- U6: Manufacturer (none) -> Texas Instruments
Connections:
- net LED_PWR: now also R138.2; no longer P2.2 (Pin_2)
- new net: P2.2 (Pin_2), R138.1

Commit message: updated per review, improved docs
Parts:
- removed R138: 0, Resistor_SMD:R_0603_1608Metric, symbol Device:R_US
- added JP1 (x3): Wire Cut Jumper, Resistor_SMD:R_0603_1608Metric, symbol Jumper:Jumper_2_Bridged
- renumbered Q69 to Q70
Connections:
- net +5V: now also JP1.2 (B); no longer P2.1 (Pin_1)
- net LED_PWR: now also JP1.2 (B)
- net NeoPixel_DIN: now also JP1.1 (A); no longer R17.2, R17.2
- net at P2.2 (Pin_2): now also JP1.1 (A)
- new net: JP1.2 (B), R17.2, R17.2
- new net: JP1.1 (A), P2.1 (Pin_1)
Other:
- note added: "cut for flight"
- moved on the sheet: R269
