File: revC-fm/low_inhibit.kicad_sch (KiCad schematic)
At the start: 14 parts, among them Q2 MMDT2907AQ, Q55 MMDT3946, Q56 BSZ025N04LSATMA1, Q57 BSZ025N04LSATMA1

Commit message: almost done!!!!!
Parts:
- D21: value D -> 1SS400T1G
- Q56, Q57: value BSZ025N04LSATMA1 -> BSZ025; Mfr. Part No BSZ025N04LS -> BSZ025N04LSATMA1
Connections:
- net at C36.1, D21.2 (A), R238.2: now also R239.2, R240.2; no longer R239.1, R240.1
- net at Q56.4 (G): now also R239.1; no longer R239.2
- net at Q57.4 (G): now also R240.1; no longer R240.2
- net IN_HI renamed IN
- net IN_LO renamed OUT
- net SW1 renamed ~{CTRL1}
- net SW4 renamed ~{CTRL2}
Other:
- note added: "Logic Inversion"
- note added: "Low Side Inhibit"
- note added: "Push-Pull Gate Driver"
- moved on the sheet: C36, D21, Q2A, Q55A, Q55B, Q56, Q57, R235, R236, R237, R238, R239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

Commit message: updated fab files
Parts:
- C36: Manufacturer (none) -> TDK; Mfr. Part No (none) -> CGA2B3X7R1H104K050BE
- D7: renamed from D21; Manufacturer (none) -> onsemi; Mfr. Part No (none) -> 1SS400T1G
- Q2: value MMDT2907AQ -> MMDT5551-7-F; Manufacturer (none) -> Diodes Incorporated; Mfr. Part No MMDT2907AQ-7-F -> MMDT5551-7-F
- Q27: renamed from Q55; Manufacturer (none) -> Diodes Incorporated
- Q28: renamed from Q56; Manufacturer (none) -> Infineon
- Q29: renamed from Q57; Manufacturer (none) -> Infineon
- R113: renamed from R235; Manufacturer (none) -> Stackpole Electronics; Mfr. Part No (none) -> RMCF0603ZT0R00
- R114: renamed from R236; Manufacturer (none) -> Stackpole Electronics; Mfr. Part No (none) -> RMCF0402FT1M00
- R115: renamed from R237; Manufacturer (none) -> Stackpole Electronics; Mfr. Part No (none) -> RMCF0402FT1M00
- R116: renamed from R238; Manufacturer (none) -> Stackpole Electronics; Mfr. Part No (none) -> RMCF0402FT220K
- R117: renamed from R241; Manufacturer (none) -> Stackpole Electronics; Mfr. Part No (none) -> RMCF0402FT1M00
- R118: renamed from R240; Manufacturer (none) -> Panasonic; Mfr. Part No (none) -> ERJ-2GEJ102X
- R119: renamed from R239; Manufacturer (none) -> Panasonic; Mfr. Part No (none) -> ERJ-2GEJ102X

Commit message: updated per review, improved docs
Parts:
- renumbered R113 to R117, R114 to R118, R115 to R119, R116 to R120, R117 to R121, R118 to R122, R119 to R123
