File: revC-fm/usb_bus_inhibit.kicad_sch (KiCad schematic)
At the start: 8 parts, among them Q22 BSZ180P03NS3GATMA1, Q23 BSZ180P03NS3GATMA1

Commit message: almost done!!!!!
Parts:
- Q22, Q23: value BSZ180P03NS3GATMA1 -> BSZ180
Connections:
- net IN_LO is gone; now on an unnamed net: Q23.1 (S), R54.2
- net at Q22.1 (S): no longer Q23.5 (D)
- net IN_HI renamed IN
- net SW4 renamed ~{CTRL}
- new net OUT: Q23.5 (D)
Other:
- note added: "USB Bus Inhibit"
- note removed: "Used for evaluation NEVER turns on during flight."
- note removed: "VBUS_USB Inhibit"
- moved on the sheet: C36, Q22, Q23, R141, R54, R57, R87

Commit message: updated fab files
Parts:
- C36: Manufacturer (none) -> TDK; Mfr. Part No (none) -> CGA2B3X7R1H104K050BE
- Q22, Q23: Manufacturer (none) -> Infineon
- R141, R87: Manufacturer (none) -> Panasonic; Mfr. Part No (none) -> ERJ-2GEJ102X
- R54, R57: Manufacturer (none) -> Stackpole Electronics; Mfr. Part No (none) -> RMCF0603ZT0R00
- R57: Manufacturer (none) -> Stackpole Electronics; Mfr. Part No (none) -> RMCF0402FT1M00
Changed lines of the file:
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@@
       (effects (font (size 1.27 1.27)) hide)
     )
-    (property "Datasheet" "~" (at 166.37 72.39 0)
+    (property "Datasheet" "https://www.infineon.com/dgdl/Infineon-BSZ180P03NS3_G-DS-v02_01-en.pdf?fileId=db3a304326dfb13001271f04398f4ec1" (at 166.37 72.39 0)
       (effects (font (size 1.27 1.27)) hide)
     )
     (property "Mfr. Part No" "BSZ180P03NS3GATMA1" (at 165.1 81.28 0)
+      (effects (font (size 1.27 1.27)) hide)
+    )
+    (property "Manufacturer" "Infineon" (at 165.1 81.28 0)
       (effects (font (size 1.27 1.27)) hide)
     )
@@
         )
         (path "/d1441985-7b63-4bf8-a06d-c70da2e3b78b/00000000-0000-0000-0000-00005cec5dde/185dd961-1d17-4f06-b36f-81ebbaab9526"
-          (reference "Q13") (unit 1)
+          (reference "Q15") (unit 1)
         )
       )
@@
       (effects (font (size 1.27 1.27)) hide)
     )
+    (property "Manufacturer" "Stackpole Electronics" (at 154.94 111.76 0)
+      (effects (font (size 1.27 1.27)) hide)
+    )
+    (property "Mfr. Part No" "RMCF0603ZT0R00" (at 154.94 111.76 0)
+      (effects (font (size 1.27 1.27)) hide)
+    )
     (pin "1")
     (pin "2")
@@
         )
         (path "/d1441985-7b63-4bf8-a06d-c70da2e3b78b/00000000-0000-0000-0000-00005cec5dde/185dd961-1d17-4f06-b36f-81ebbaab9526"
-          (reference "R68") (unit 1)
+          (reference "R94") (unit 1)
         )
       )
@@
       (effects (font (size 1.27 1.27)) hide)
     )
-    (property "Mfr. Part No" "" (at 146.05 92.71 0)
+    (property "Mfr. Part No" "ERJ-2GEJ102X" (at 146.05 92.71 0)
+      (effects (font (size 1.27 1.27)) hide)
+    )
+    (property "Manufacturer" "Panasonic" (at 146.05 92.71 0)
       (effects (font (size 1.27 1.27)) hide)
     )
@@
         )
         (path "/d1441985-7b63-4bf8-a06d-c70da2e3b78b/00000000-0000-0000-0000-00005cec5dde/185dd961-1d17-4f06-b36f-81ebbaab9526"
-          (reference "R69") (unit 1)
+          (reference "R92") (unit 1)
         )
       )
@@
       (effects (font (size 1.27 1.27)) hide)
     )
-    (property "Mfr. Part No" "" (at 154.94 130.81 0)
+    (property "Mfr. Part No" "RMCF0402FT1M00" (at 154.94 130.81 0)
+      (effects (font (size 1.27 1.27)) hide)
+    )
+    (property "Manufacturer" "Stackpole Electronics" (at 154.94 130.81 0)
       (effects (font (size 1.27 1.27)) hide)
     )
@@
         )
         (path "/d1441985-7b63-4bf8-a06d-c70da2e3b78b/00000000-0000-0000-0000-00005cec5dde/185dd961-1d17-4f06-b36f-81ebbaab9526"
-          (reference "R71") (unit 1)
+          (reference "R95") (unit 1)
         )
       )
@@
       (effects (font (size 1.27 1.27)) hide)
     )
-    (property "Datasheet" "~" (at 144.78 72.39 0)
+    (property "Datasheet" "https://www.infineon.com/dgdl/Infineon-BSZ180P03NS3_G-DS-v02_01-en.pdf?fileId=db3a304326dfb13001271f04398f4ec1" (at 144.78 72.39 0)
       (effects (font (size 1.27 1.27)) hide)
     )
     (property "Mfr. Part No" "BSZ180P03NS3GATMA1" (at 146.05 81.28 0)
+      (effects (font (size 1.27 1.27)) hide)
+    )
+    (property "Manufacturer" "Infineon" (at 146.05 81.28 0)
       (effects (font (size 1.27 1.27)) hide)
     )
@@
         )
         (path "/d1441985-7b63-4bf8-a06d-c70da2e3b78b/00000000-0000-0000-0000-00005cec5dde/185dd961-1d17-4f06-b36f-81ebbaab9526"
-          (reference "Q12") (unit 1)
+          (reference "Q14") (unit 1)
         )
       )
@@
       (effects (font (size 1.27 1.27)) hide)
     )
-    (property "Mfr. Part No" "" (at 114.3 139.7 0)
+    (property "Mfr. Part No" "RMCF0603ZT0R00" (at 114.3 139.7 0)
+      (effects (font (size 1.27 1.27)) hide)
+    )
+    (property "Manufacturer" "Stackpole Electronics" (at 114.3 139.7 0)
       (effects (font (size 1.27 1.27)) hide)
     )
@@
         )
         (path "/d1441985-7b63-4bf8-a06d-c70da2e3b78b/00000000-0000-0000-0000-00005cec5dde/185dd961-1d17-4f06-b36f-81ebbaab9526"
-          (reference "R72") (unit 1)
+          (reference "R96") (unit 1)
         )
       )
@@
       (effects (font (size 1.27 1.27)) hide)
     )
-    (property "Mfr. Part No" "" (at 165.1 92.71 0)
+    (property "Mfr. Part No" "ERJ-2GEJ102X" (at 165.1 92.71 0)
+      (effects (font (size 1.27 1.27)) hide)
+    )
+    (property "Manufacturer" "Panasonic" (at 165.1 92.71 0)
       (effects (font (size 1.27 1.27)) hide)
     )
@@
         )
         (path "/d1441985-7b63-4bf8-a06d-c70da2e3b78b/00000000-0000-0000-0000-00005cec5dde/185dd961-1d17-4f06-b36f-81ebbaab9526"
-          (reference "R70") (unit 1)
+          (reference "R93") (unit 1)
         )
       )
@@
       (effects (font (size 1.27 1.27)) hide)
     )
-    (property "Mfr. Part No" "" (at 165.1 130.81 0)
+    (property "Mfr. Part No" "CGA2B3X7R1H104K050BE" (at 165.1 130.81 0)
+      (effects (font (size 1.27 1.27)) hide)
+    )
+    (property "Manufacturer" "TDK" (at 165.1 130.81 0)
       (effects (font (size 1.27 1.27)) hide)
     )
@@
         )
         (path "/d1441985-7b63-4bf8-a06d-c70da2e3b78b/00000000-0000-0000-0000-00005cec5dde/185dd961-1d17-4f06-b36f-81ebbaab9526"
-          (reference "C54") (unit 1)
-        )
-      )
+          (reference "C56") (unit 1)
+        )
+      )

Commit message: updated per review, improved docs
Parts:
- R57: value 1Meg -> 220k; Mfr. Part No RMCF0402FT1M00 -> RMCF0402FT220K
Changed lines of the file:
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@@
+    (stroke (width 0) (type default))
+  )
+  (wire (pts (xy 91.44 81.28) (xy 140.97 81.28))
     (stroke (width 0) (type default))
   )
@@
   )
   (wire (pts (xy 170.18 81.28) (xy 208.28 81.28))
-    (stroke (width 0) (type default))
-  )
-  (wire (pts (xy 91.44 81.28) (xy 140.97 81.28))
     (stroke (width 0) (type default))
   )
@@
       (effects (font (size 1.27 1.27)) hide)
     )
+    (property "Description" "MOSFET P-CH 30V 9A/39.6A TSDSON" (at 165.1 81.28 0)
+      (effects (font (size 1.27 1.27)) hide)
+    )
     (pin "1")
     (pin "4")
@@
       (effects (font (size 1.27 1.27)) hide)
     )
+    (property "Description" "RES 0 OHM JUMPER 1/10W 0603" (at 154.94 111.76 0)
+      (effects (font (size 1.27 1.27)) hide)
+    )
     (pin "1")
     (pin "2")
@@
         )
         (path "/d1441985-7b63-4bf8-a06d-c70da2e3b78b/00000000-0000-0000-0000-00005cec5dde/185dd961-1d17-4f06-b36f-81ebbaab9526"
-          (reference "R94") (unit 1)
+          (reference "R98") (unit 1)
         )
       )
@@
       (effects (font (size 1.27 1.27)) hide)
     )
+    (property "Description" "RES SMD 1K OHM 5% 1/10W 0402" (at 146.05 92.71 0)
+      (effects (font (size 1.27 1.27)) hide)
+    )
     (pin "1")
     (pin "2")
@@
         )
         (path "/d1441985-7b63-4bf8-a06d-c70da2e3b78b/00000000-0000-0000-0000-00005cec5dde/185dd961-1d17-4f06-b36f-81ebbaab9526"
-          (reference "R92") (unit 1)
+          (reference "R96") (unit 1)
         )
       )
@@
       (effects (font (size 1.27 1.27)) (justify left))
     )
-    (property "Value" "1Meg" (at 156.6672 131.953 0)
+    (property "Value" "220k" (at 156.6672 131.953 0)
       (effects (font (size 1.27 1.27)) (justify left))
     )
@@
       (effects (font (size 1.27 1.27)) hide)
     )
-    (property "Mfr. Part No" "RMCF0402FT1M00" (at 154.94 130.81 0)
+    (property "Mfr. Part No" "RMCF0402FT220K" (at 154.94 130.81 0)
       (effects (font (size 1.27 1.27)) hide)
     )
@@
       (effects (font (size 1.27 1.27)) hide)
     )
+    (property "Description" "RES 220K OHM 1% 1/16W 0402" (at 154.94 130.81 0)
+      (effects (font (size 1.27 1.27)) hide)
+    )
     (pin "1")
     (pin "2")
@@
         )
         (path "/d1441985-7b63-4bf8-a06d-c70da2e3b78b/00000000-0000-0000-0000-00005cec5dde/185dd961-1d17-4f06-b36f-81ebbaab9526"
-          (reference "R95") (unit 1)
+          (reference "R99") (unit 1)
         )
       )
@@
       (effects (font (size 1.27 1.27)) hide)
     )
+    (property "Description" "MOSFET P-CH 30V 9A/39.6A TSDSON" (at 146.05 81.28 0)
+      (effects (font (size 1.27 1.27)) hide)
+    )
     (pin "1")
     (pin "4")
@@
       (effects (font (size 1.27 1.27)) hide)
     )
+    (property "Description" "RES 0 OHM JUMPER 1/10W 0603" (at 114.3 139.7 0)
+      (effects (font (size 1.27 1.27)) hide)
+    )
     (pin "1")
     (pin "2")
@@
         )
         (path "/d1441985-7b63-4bf8-a06d-c70da2e3b78b/00000000-0000-0000-0000-00005cec5dde/185dd961-1d17-4f06-b36f-81ebbaab9526"
-          (reference "R96") (unit 1)
+          (reference "R100") (unit 1)
         )
       )
@@
       (effects (font (size 1.27 1.27)) hide)
     )
+    (property "Description" "RES SMD 1K OHM 5% 1/10W 0402" (at 165.1 92.71 0)
+      (effects (font (size 1.27 1.27)) hide)
+    )
     (pin "1")
     (pin "2")
@@
         )
         (path "/d1441985-7b63-4bf8-a06d-c70da2e3b78b/00000000-0000-0000-0000-00005cec5dde/185dd961-1d17-4f06-b36f-81ebbaab9526"
-          (reference "R93") (unit 1)
+          (reference "R97") (unit 1)
         )
       )
@@
       (effects (font (size 1.27 1.27)) hide)
     )
+    (property "Description" "CAP CER 0.1UF 50V X7R 0402" (at 165.1 130.81 0)
+      (effects (font (size 1.27 1.27)) hide)
+    )
     (pin "1")
     (pin "2")
@@
         )
         (path "/d1441985-7b63-4bf8-a06d-c70da2e3b78b/00000000-0000-0000-0000-00005cec5dde/185dd961-1d17-4f06-b36f-81ebbaab9526"
-          (reference "C56") (unit 1)
-        )
-      )
+          (reference "C57") (unit 1)
+        )
+      )
