File: revC-fm/usb_chrg_inhibit.kicad_sch (KiCad schematic)
At the start: 9 parts, among them Q21 MMDT3946, Q22 BSZ180P03NS3GATMA1, Q23 BSZ180P03NS3GATMA1

Commit message: almost done!!!!!
Parts:
- Q22, Q23: value BSZ180P03NS3GATMA1 -> BSZ180
Connections:
- net IN_LO is gone; now on an unnamed net: Q23.1 (S), R54.2
- net at Q22.1 (S): no longer Q23.5 (D)
- net at Q21.2 (B1): now also R57.1; no longer R57.2
- net IN_HI renamed IN
- net IN: now also R57.2; no longer R57.1
- net ~{RBF} renamed ~{CTRL}
- new net OUT: Q23.5 (D)
Other:
- note added: "USB Charge Inhibit"
- note removed: "Closed when RBF IN & 5V_USB"
- note removed: "Used for ground charge. NEVER turns on during flight."
- note removed: "VCHRG_USB Inhibit"
- moved on the sheet: C36, Q21A, Q21B, Q22, Q23, R141, R54, R57, R87

Commit message: updated fab files
Parts:
- C36: Manufacturer (none) -> TDK; Mfr. Part No (none) -> CGA2B3X7R1H104K050BE
- Q21: Manufacturer (none) -> Diodes Incorporated
- Q22, Q23: Manufacturer (none) -> Infineon
- R141, R87: Manufacturer (none) -> Panasonic; Mfr. Part No (none) -> ERJ-2GEJ102X
- R54: Manufacturer (none) -> Stackpole Electronics; Mfr. Part No (none) -> RMCF0603ZT0R00
- R57: Manufacturer (none) -> Stackpole Electronics; Mfr. Part No (none) -> RMCF0402FT100K
- R57: Manufacturer (none) -> Stackpole Electronics; Mfr. Part No (none) -> RMCF0402FT1M00
Changed lines of the file:
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@@
       (effects (font (size 1.27 1.27)) hide)
     )
-    (property "Datasheet" "~" (at 157.48 64.77 0)
+    (property "Datasheet" "https://www.infineon.com/dgdl/Infineon-BSZ180P03NS3_G-DS-v02_01-en.pdf?fileId=db3a304326dfb13001271f04398f4ec1" (at 157.48 64.77 0)
       (effects (font (size 1.27 1.27)) hide)
     )
     (property "Mfr. Part No" "BSZ180P03NS3GATMA1" (at 158.75 73.66 0)
+      (effects (font (size 1.27 1.27)) hide)
+    )
+    (property "Manufacturer" "Infineon" (at 158.75 73.66 0)
       (effects (font (size 1.27 1.27)) hide)
     )
@@
         )
         (path "/d1441985-7b63-4bf8-a06d-c70da2e3b78b/00000000-0000-0000-0000-00005cec5dde/4c3121c8-bd10-459a-a6ea-38d5e9e20bca"
-          (reference "Q8") (unit 1)
+          (reference "Q11") (unit 1)
         )
         (path "/d1441985-7b63-4bf8-a06d-c70da2e3b78b/00000000-0000-0000-0000-00005cec5dde/185dd961-1d17-4f06-b36f-81ebbaab9526"
@@
         )
         (path "/d1441985-7b63-4bf8-a06d-c70da2e3b78b/00000000-0000-0000-0000-00005cec5dde/4c3121c8-bd10-459a-a6ea-38d5e9e20bca"
-          (reference "#PWR089") (unit 1)
+          (reference "#PWR0102") (unit 1)
         )
         (path "/d1441985-7b63-4bf8-a06d-c70da2e3b78b/00000000-0000-0000-0000-00005cec5dde/185dd961-1d17-4f06-b36f-81ebbaab9526"
@@
       (effects (font (size 1.27 1.27)) hide)
     )
-    (property "Mfr. Part No" "" (at 176.53 85.09 0)
+    (property "Mfr. Part No" "ERJ-2GEJ102X" (at 176.53 85.09 0)
+      (effects (font (size 1.27 1.27)) hide)
+    )
+    (property "Manufacturer" "Panasonic" (at 176.53 85.09 0)
       (effects (font (size 1.27 1.27)) hide)
     )
@@
         )
         (path "/d1441985-7b63-4bf8-a06d-c70da2e3b78b/00000000-0000-0000-0000-00005cec5dde/4c3121c8-bd10-459a-a6ea-38d5e9e20bca"
-          (reference "R64") (unit 1)
+          (reference "R89") (unit 1)
         )
         (path "/d1441985-7b63-4bf8-a06d-c70da2e3b78b/00000000-0000-0000-0000-00005cec5dde/185dd961-1d17-4f06-b36f-81ebbaab9526"
@@
     )
     (property "Mfr. Part No" "MMDT3946-7-F" (at 156.21 120.65 0)
+      (effects (font (size 1.27 1.27)) hide)
+    )
+    (property "Manufacturer" "Diodes Incorporated" (at 156.21 120.65 0)
       (effects (font (size 1.27 1.27)) hide)
     )
@@
         )
         (path "/d1441985-7b63-4bf8-a06d-c70da2e3b78b/00000000-0000-0000-0000-00005cec5dde/4c3121c8-bd10-459a-a6ea-38d5e9e20bca"
-          (reference "Q10") (unit 1)
+          (reference "Q13") (unit 1)
         )
         (path "/d1441985-7b63-4bf8-a06d-c70da2e3b78b/00000000-0000-0000-0000-00005cec5dde/185dd961-1d17-4f06-b36f-81ebbaab9526"
@@
       (effects (font (size 1.27 1.27)) hide)
     )
-    (property "Mfr. Part No" "" (at 158.75 85.09 0)
+    (property "Mfr. Part No" "ERJ-2GEJ102X" (at 158.75 85.09 0)
+      (effects (font (size 1.27 1.27)) hide)
+    )
+    (property "Manufacturer" "Panasonic" (at 158.75 85.09 0)
       (effects (font (size 1.27 1.27)) hide)
     )
@@
         )
         (path "/d1441985-7b63-4bf8-a06d-c70da2e3b78b/00000000-0000-0000-0000-00005cec5dde/4c3121c8-bd10-459a-a6ea-38d5e9e20bca"
-          (reference "R63") (unit 1)
+          (reference "R88") (unit 1)
         )
         (path "/d1441985-7b63-4bf8-a06d-c70da2e3b78b/00000000-0000-0000-0000-00005cec5dde/185dd961-1d17-4f06-b36f-81ebbaab9526"
@@
       (effects (font (size 1.27 1.27)) hide)
     )
-    (property "Mfr. Part No" "" (at 146.05 105.41 0)
+    (property "Mfr. Part No" "RMCF0402FT100K" (at 146.05 105.41 0)
+      (effects (font (size 1.27 1.27)) hide)
+    )
+    (property "Manufacturer" "Stackpole Electronics" (at 146.05 105.41 0)
       (effects (font (size 1.27 1.27)) hide)
     )
@@
         )
         (path "/d1441985-7b63-4bf8-a06d-c70da2e3b78b/00000000-0000-0000-0000-00005cec5dde/4c3121c8-bd10-459a-a6ea-38d5e9e20bca"
-          (reference "R66") (unit 1)
+          (reference "R90") (unit 1)
         )
         (path "/d1441985-7b63-4bf8-a06d-c70da2e3b78b/00000000-0000-0000-0000-00005cec5dde/185dd961-1d17-4f06-b36f-81ebbaab9526"
@@
       (effects (font (size 1.27 1.27)) hide)
     )
-    (property "Mfr. Part No" "" (at 176.53 105.41 0)
+    (property "Mfr. Part No" "CGA2B3X7R1H104K050BE" (at 176.53 105.41 0)
+      (effects (font (size 1.27 1.27)) hide)
+    )
+    (property "Manufacturer" "TDK" (at 176.53 105.41 0)
       (effects (font (size 1.27 1.27)) hide)
     )
@@
         )
         (path "/d1441985-7b63-4bf8-a06d-c70da2e3b78b/00000000-0000-0000-0000-00005cec5dde/4c3121c8-bd10-459a-a6ea-38d5e9e20bca"
-          (reference "C53") (unit 1)
+          (reference "C55") (unit 1)
         )
         (path "/d1441985-7b63-4bf8-a06d-c70da2e3b78b/00000000-0000-0000-0000-00005cec5dde/185dd961-1d17-4f06-b36f-81ebbaab9526"
@@
       (effects (font (size 1.27 1.27)) hide)
     )
-    (property "Datasheet" "~" (at 177.8 64.77 0)
+    (property "Datasheet" "https://www.infineon.com/dgdl/Infineon-BSZ180P03NS3_G-DS-v02_01-en.pdf?fileId=db3a304326dfb13001271f04398f4ec1" (at 177.8 64.77 0)
       (effects (font (size 1.27 1.27)) hide)
     )
     (property "Mfr. Part No" "BSZ180P03NS3GATMA1" (at 176.53 73.66 0)
+      (effects (font (size 1.27 1.27)) hide)
+    )
+    (property "Manufacturer" "Infineon" (at 176.53 73.66 0)
       (effects (font (size 1.27 1.27)) hide)
     )
@@
         )
         (path "/d1441985-7b63-4bf8-a06d-c70da2e3b78b/00000000-0000-0000-0000-00005cec5dde/4c3121c8-bd10-459a-a6ea-38d5e9e20bca"
-          (reference "Q9") (unit 1)
+          (reference "Q12") (unit 1)
         )
         (path "/d1441985-7b63-4bf8-a06d-c70da2e3b78b/00000000-0000-0000-0000-00005cec5dde/185dd961-1d17-4f06-b36f-81ebbaab9526"
@@
       (effects (font (size 1.27 1.27)) hide)
     )
+    (property "Manufacturer" "Stackpole Electronics" (at 167.64 82.55 0)
+      (effects (font (size 1.27 1.27)) hide)
+    )
+    (property "Mfr. Part No" "RMCF0603ZT0R00" (at 167.64 82.55 0)
+      (effects (font (size 1.27 1.27)) hide)
+    )
     (pin "1")
     (pin "2")
@@
         )
         (path "/d1441985-7b63-4bf8-a06d-c70da2e3b78b/00000000-0000-0000-0000-00005cec5dde/4c3121c8-bd10-459a-a6ea-38d5e9e20bca"
-          (reference "R62") (unit 1)
+          (reference "R87") (unit 1)
         )
         (path "/d1441985-7b63-4bf8-a06d-c70da2e3b78b/00000000-0000-0000-0000-00005cec5dde/185dd961-1d17-4f06-b36f-81ebbaab9526"
@@
       (effects (font (size 1.27 1.27)) hide)
     )
-    (property "Mfr. Part No" "" (at 167.64 105.41 0)
+    (property "Mfr. Part No" "RMCF0402FT1M00" (at 167.64 105.41 0)
+      (effects (font (size 1.27 1.27)) hide)
+    )
+    (property "Manufacturer" "Stackpole Electronics" (at 167.64 105.41 0)
       (effects (font (size 1.27 1.27)) hide)
     )
@@
         )
         (path "/d1441985-7b63-4bf8-a06d-c70da2e3b78b/00000000-0000-0000-0000-00005cec5dde/4c3121c8-bd10-459a-a6ea-38d5e9e20bca"
-          (reference "R65") (unit 1)
+          (reference "R91") (unit 1)
         )
         (path "/d1441985-7b63-4bf8-a06d-c70da2e3b78b/00000000-0000-0000-0000-00005cec5dde/185dd961-1d17-4f06-b36f-81ebbaab9526"
@@
     )
     (property "Mfr. Part No" "MMDT3946-7-F" (at 156.21 130.81 0)
+      (effects (font (size 1.27 1.27)) hide)
+    )
+    (property "Manufacturer" "Diodes Incorporated" (at 156.21 130.81 0)
       (effects (font (size 1.27 1.27)) hide)
     )
@@
         )
         (path "/d1441985-7b63-4bf8-a06d-c70da2e3b78b/00000000-0000-0000-0000-00005cec5dde/4c3121c8-bd10-459a-a6ea-38d5e9e20bca"
-          (reference "Q10") (unit 2)
-        )
-        (path "/d1441985-7b63-4bf8-a06d-c70da2e3b78b/00000000-0000-0000-0000-00005cec5dde/185dd961-1d17-4f06-b36f-81ebbaab9526"
+          (reference "Q13") (unit 2)
+        )
+        (path "/d1441985-7b63-4bf8-a06d-c70da2e3b78b/00000000-0000-0000-0000-00005cec5dde/185dd961-1d17-4f06-b36f-81ebbaab9526"

Commit message: updated per review, improved docs
Parts:
- R57: value 1Meg -> 220k; Mfr. Part No RMCF0402FT1M00 -> RMCF0402FT220K
Changed lines of the file:
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@@
+    (stroke (width 0) (type default))
+  )
+  (wire (pts (xy 158.75 114.3) (xy 167.64 114.3))
+    (stroke (width 0) (type default))
+  )
+  (wire (pts (xy 158.75 114.3) (xy 158.75 115.57))
+    (stroke (width 0) (type default))
+  )
+  (wire (pts (xy 167.64 97.79) (xy 167.64 101.6))
+    (stroke (width 0) (type default))
+  )
+  (wire (pts (xy 158.75 91.44) (xy 176.53 91.44))
+    (stroke (width 0) (type default))
+  )
+  (wire (pts (xy 100.33 130.81) (xy 151.13 130.81))
+    (stroke (width 0) (type default))
+  )
+  (wire (pts (xy 176.53 97.79) (xy 176.53 101.6))
+    (stroke (width 0) (type default))
+  )
+  (wire (pts (xy 146.05 73.66) (xy 146.05 101.6))
+    (stroke (width 0) (type default))
+  )
+  (wire (pts (xy 181.61 73.66) (xy 217.17 73.66))
+    (stroke (width 0) (type default))
+  )
+  (wire (pts (xy 158.75 135.89) (xy 158.75 138.43))
+    (stroke (width 0) (type default))
+  )
+  (wire (pts (xy 158.75 91.44) (xy 158.75 114.3))
+    (stroke (width 0) (type default))
+  )
+  (wire (pts (xy 176.53 91.44) (xy 176.53 88.9))
+    (stroke (width 0) (type default))
+  )
+  (wire (pts (xy 167.64 109.22) (xy 167.64 114.3))
+    (stroke (width 0) (type default))
+  )
+  (wire (pts (xy 176.53 109.22) (xy 176.53 114.3))
+    (stroke (width 0) (type default))
+  )
+  (wire (pts (xy 167.64 97.79) (xy 167.64 86.36))
+    (stroke (width 0) (type default))
+  )
+  (wire (pts (xy 163.83 73.66) (xy 167.64 73.66))
+    (stroke (width 0) (type default))
+  )
+  (wire (pts (xy 176.53 114.3) (xy 167.64 114.3))
     (stroke (width 0) (type default))
   )
   (wire (pts (xy 100.33 73.66) (xy 146.05 73.66))
-    (stroke (width 0) (type default))
-  )
-  (wire (pts (xy 158.75 114.3) (xy 167.64 114.3))
-    (stroke (width 0) (type default))
-  )
-  (wire (pts (xy 158.75 114.3) (xy 158.75 115.57))
-    (stroke (width 0) (type default))
-  )
-  (wire (pts (xy 167.64 97.79) (xy 167.64 101.6))
-    (stroke (width 0) (type default))
-  )
-  (wire (pts (xy 158.75 91.44) (xy 176.53 91.44))
-    (stroke (width 0) (type default))
-  )
-  (wire (pts (xy 100.33 130.81) (xy 151.13 130.81))
-    (stroke (width 0) (type default))
-  )
-  (wire (pts (xy 176.53 97.79) (xy 176.53 101.6))
-    (stroke (width 0) (type default))
-  )
-  (wire (pts (xy 146.05 73.66) (xy 146.05 101.6))
-    (stroke (width 0) (type default))
-  )
-  (wire (pts (xy 181.61 73.66) (xy 217.17 73.66))
-    (stroke (width 0) (type default))
-  )
-  (wire (pts (xy 158.75 135.89) (xy 158.75 138.43))
-    (stroke (width 0) (type default))
-  )
-  (wire (pts (xy 158.75 91.44) (xy 158.75 114.3))
-    (stroke (width 0) (type default))
-  )
-  (wire (pts (xy 176.53 91.44) (xy 176.53 88.9))
-    (stroke (width 0) (type default))
-  )
-  (wire (pts (xy 167.64 109.22) (xy 167.64 114.3))
-    (stroke (width 0) (type default))
-  )
-  (wire (pts (xy 176.53 109.22) (xy 176.53 114.3))
-    (stroke (width 0) (type default))
-  )
-  (wire (pts (xy 167.64 97.79) (xy 167.64 86.36))
-    (stroke (width 0) (type default))
-  )
-  (wire (pts (xy 163.83 73.66) (xy 167.64 73.66))
-    (stroke (width 0) (type default))
-  )
-  (wire (pts (xy 176.53 114.3) (xy 167.64 114.3))
     (stroke (width 0) (type default))
   )
@@
       (effects (font (size 1.27 1.27)) hide)
     )
+    (property "Description" "MOSFET P-CH 30V 9A/39.6A TSDSON" (at 158.75 73.66 0)
+      (effects (font (size 1.27 1.27)) hide)
+    )
     (pin "1")
     (pin "4")
@@
         )
         (path "/d1441985-7b63-4bf8-a06d-c70da2e3b78b/00000000-0000-0000-0000-00005cec5dde/4c3121c8-bd10-459a-a6ea-38d5e9e20bca"
-          (reference "#PWR0102") (unit 1)
+          (reference "#PWR0107") (unit 1)
         )
         (path "/d1441985-7b63-4bf8-a06d-c70da2e3b78b/00000000-0000-0000-0000-00005cec5dde/185dd961-1d17-4f06-b36f-81ebbaab9526"
@@
       (effects (font (size 1.27 1.27)) hide)
     )
+    (property "Description" "RES SMD 1K OHM 5% 1/10W 0402" (at 176.53 85.09 0)
+      (effects (font (size 1.27 1.27)) hide)
+    )
     (pin "1")
     (pin "2")
@@
         )
         (path "/d1441985-7b63-4bf8-a06d-c70da2e3b78b/00000000-0000-0000-0000-00005cec5dde/4c3121c8-bd10-459a-a6ea-38d5e9e20bca"
-          (reference "R89") (unit 1)
+          (reference "R93") (unit 1)
         )
         (path "/d1441985-7b63-4bf8-a06d-c70da2e3b78b/00000000-0000-0000-0000-00005cec5dde/185dd961-1d17-4f06-b36f-81ebbaab9526"
@@
     )
     (property "Manufacturer" "Diodes Incorporated" (at 156.21 120.65 0)
+      (effects (font (size 1.27 1.27)) hide)
+    )
+    (property "Description" "TRANS NPN/PNP 40V 0.2A SOT363" (at 156.21 120.65 0)
       (effects (font (size 1.27 1.27)) hide)
     )
@@
       (effects (font (size 1.27 1.27)) hide)
     )
+    (property "Description" "RES SMD 1K OHM 5% 1/10W 0402" (at 158.75 85.09 0)
+      (effects (font (size 1.27 1.27)) hide)
+    )
     (pin "1")
     (pin "2")
@@
         )
         (path "/d1441985-7b63-4bf8-a06d-c70da2e3b78b/00000000-0000-0000-0000-00005cec5dde/4c3121c8-bd10-459a-a6ea-38d5e9e20bca"
-          (reference "R88") (unit 1)
+          (reference "R92") (unit 1)
         )
         (path "/d1441985-7b63-4bf8-a06d-c70da2e3b78b/00000000-0000-0000-0000-00005cec5dde/185dd961-1d17-4f06-b36f-81ebbaab9526"
@@
       (effects (font (size 1.27 1.27)) hide)
     )
+    (property "Description" "RES 100K OHM 1% 1/16W 0402" (at 146.05 105.41 0)
+      (effects (font (size 1.27 1.27)) hide)
+    )
     (pin "1")
     (pin "2")
@@
         )
         (path "/d1441985-7b63-4bf8-a06d-c70da2e3b78b/00000000-0000-0000-0000-00005cec5dde/4c3121c8-bd10-459a-a6ea-38d5e9e20bca"
-          (reference "R90") (unit 1)
+          (reference "R94") (unit 1)
         )
         (path "/d1441985-7b63-4bf8-a06d-c70da2e3b78b/00000000-0000-0000-0000-00005cec5dde/185dd961-1d17-4f06-b36f-81ebbaab9526"
@@
     )
     (property "Manufacturer" "TDK" (at 176.53 105.41 0)
+      (effects (font (size 1.27 1.27)) hide)
+    )
+    (property "Description" "CAP CER 0.1UF 50V X7R 0402" (at 176.53 105.41 0)
       (effects (font (size 1.27 1.27)) hide)
     )
@@
         )
         (path "/d1441985-7b63-4bf8-a06d-c70da2e3b78b/00000000-0000-0000-0000-00005cec5dde/4c3121c8-bd10-459a-a6ea-38d5e9e20bca"
-          (reference "C55") (unit 1)
+          (reference "C56") (unit 1)
         )
         (path "/d1441985-7b63-4bf8-a06d-c70da2e3b78b/00000000-0000-0000-0000-00005cec5dde/185dd961-1d17-4f06-b36f-81ebbaab9526"
@@
       (effects (font (size 1.27 1.27)) hide)
     )
+    (property "Description" "MOSFET P-CH 30V 9A/39.6A TSDSON" (at 176.53 73.66 0)
+      (effects (font (size 1.27 1.27)) hide)
+    )
     (pin "1")
     (pin "4")
@@
       (effects (font (size 1.27 1.27)) hide)
     )
+    (property "Description" "RES 0 OHM JUMPER 1/10W 0603" (at 167.64 82.55 0)
+      (effects (font (size 1.27 1.27)) hide)
+    )
     (pin "1")
     (pin "2")
@@
         )
         (path "/d1441985-7b63-4bf8-a06d-c70da2e3b78b/00000000-0000-0000-0000-00005cec5dde/4c3121c8-bd10-459a-a6ea-38d5e9e20bca"
-          (reference "R87") (unit 1)
+          (reference "R91") (unit 1)
         )
         (path "/d1441985-7b63-4bf8-a06d-c70da2e3b78b/00000000-0000-0000-0000-00005cec5dde/185dd961-1d17-4f06-b36f-81ebbaab9526"
@@
       (effects (font (size 1.27 1.27)) (justify left))
     )
-    (property "Value" "1Meg" (at 165.9128 106.553 0)
+    (property "Value" "220k" (at 165.9128 106.553 0)
       (effects (font (size 1.27 1.27)) (justify left))
     )
@@
       (effects (font (size 1.27 1.27)) hide)
     )
-    (property "Mfr. Part No" "RMCF0402FT1M00" (at 167.64 105.41 0)
+    (property "Mfr. Part No" "RMCF0402FT220K" (at 167.64 105.41 0)
       (effects (font (size 1.27 1.27)) hide)
     )
@@
       (effects (font (size 1.27 1.27)) hide)
     )
+    (property "Description" "RES 220K OHM 1% 1/16W 0402" (at 167.64 105.41 0)
+      (effects (font (size 1.27 1.27)) hide)
+    )
     (pin "1")
     (pin "2")
@@
         )
         (path "/d1441985-7b63-4bf8-a06d-c70da2e3b78b/00000000-0000-0000-0000-00005cec5dde/4c3121c8-bd10-459a-a6ea-38d5e9e20bca"
-          (reference "R91") (unit 1)
+          (reference "R95") (unit 1)
         )
         (path "/d1441985-7b63-4bf8-a06d-c70da2e3b78b/00000000-0000-0000-0000-00005cec5dde/185dd961-1d17-4f06-b36f-81ebbaab9526"
@@
       (effects (font (size 1.27 1.27)) hide)
     )
+    (property "Description" "TRANS NPN/PNP 40V 0.2A SOT363" (at 156.21 130.81 0)
+      (effects (font (size 1.27 1.27)) hide)
+    )
